Commit message: doc:1.修改stl和urdf文件设置为零位状态2.修改机械臂的限位3.修改eco656F的包名

File: ECO65/urdf/eco_65_6f_description/urdf/eco656weili.sldasm.urdf (robot description, URDF)
Before this commit: robot eco656weili.sldasm, 7 links, 6 joints
Links:
- link Link1: mass 1.5078 -> 0.74252212802658; geometry collision mesh filename=package://eco656weili/meshes/Link1.STL; visual mesh filename=package://eco656weili/meshes/Link1.STL
- link Link2: mass 2.0227 -> 1.35020712394805; geometry collision mesh filename=package://eco656weili/meshes/Link2.STL; visual mesh filename=package://eco656weili/meshes/Link2.STL
- link Link3: mass 1.8858 -> 1.0422213139163; geometry collision mesh filename=package://eco656weili/meshes/Link3.STL; visual mesh filename=package://eco656weili/meshes/Link3.STL
- link Link4: mass 0.5701 -> 0.273792481713346; geometry collision mesh filename=package://eco656weili/meshes/Link4.STL; visual mesh filename=package://eco656weili/meshes/Link4.STL
- link Link5: mass 0.6414 -> 0.27793758472494; geometry collision mesh filename=package://eco656weili/meshes/Link5.STL; visual mesh filename=package://eco656weili/meshes/Link5.STL
- link Link6: mass 0.19 -> 0.14611108984048; geometry collision mesh filename=package://eco656weili/meshes/Link6.STL; visual mesh filename=package://eco656weili/meshes/Link6.STL
- link baselink: mass 0.611273147318723 -> 0.61127; geometry collision mesh filename=package://eco656weili/meshes/base_link.STL; visual mesh filename=package://eco656weili/meshes/base_link.STL
Joints:
- removed joint joint1
- removed joint joint2
- removed joint joint3
- removed joint joint4
- removed joint joint5
- removed joint joint6
- added joint Joint1: type revolute, parent baselink, child Link1, origin xyz=0 0 0.1625 rpy=0 0 0, axis 0 0 -1, limit lower=-3.1923 upper=3.1923 effort=100 velocity=1
- added joint Joint2: type revolute, parent Link1, child Link2, origin xyz=-0.086 0 0 rpy=1.5708 0 0, axis 3.5522E-05 0 -1, limit lower=-2.61666 upper=2.442 effort=100 velocity=1
- added joint Joint3: type revolute, parent Link2, child Link3, origin xyz=0 0.26 0 rpy=3.1416 0 1.5708, axis 0 -3.5522E-05 -1, limit lower=-2.50666 upper=2.61666 effort=100 velocity=1
- added joint Joint4: type revolute, parent Link3, child Link4, origin xyz=0.24 0 -0.05888 rpy=0 0 1.5708, axis -3.5522E-05 0 -1, limit lower=-2.61666 upper=2.61666 effort=100 velocity=1
- added joint Joint5: type revolute, parent Link4, child Link5, origin xyz=0 -0.11 -1.7417E-05 rpy=1.5708 0 0, axis 0 0 -1, limit lower=-2.96555 upper=2.96555 effort=100 velocity=1
- added joint Joint6: type revolute, parent Link5, child Link6, origin xyz=0 0.108 0 rpy=-1.5708 0 0, axis -3.5522E-05 0 -1, limit lower=-2.96555 upper=2.96555 effort=100 velocity=1

File: ECO65/urdf/eco_65_b_description/urdf/eco65-2.urdf (robot description, URDF)
Before this commit: robot eco65-2, 7 links, 6 joints
Links:
- link Link6: mass 0.033842 -> 0.033025
Joints:
- joint joint1: limit lower=-3.14 upper=3.14 effort=100 velocity=1 -> lower=-3.1923 upper=3.1923 effort=100 velocity=1
- joint joint2: axis 0 0 1 -> 0 0 -1; limit lower=-3.14 upper=3.14 effort=100 velocity=1 -> lower=-2.61666 upper=2.442 effort=100 velocity=1
- joint joint3: limit lower=-2.79 upper=2.53 effort=100 velocity=1 -> lower=-2.50666 upper=2.61666 effort=100 velocity=1
- joint joint4: limit lower=-2.44 upper=2.44 effort=100 velocity=1 -> lower=-2.61666 upper=2.61666 effort=100 velocity=1; origin xyz=0 -0.24 -0.05888 rpy=0 0 1.5708 -> xyz=0.24 0 -0.05888 rpy=0 0 1.5708
- joint joint5: limit lower=-3.14 upper=3.14 effort=100 velocity=1 -> lower=-2.96555 upper=2.96555 effort=100 velocity=1; origin xyz=0 -0.11 0 rpy=1.5708 0 0 -> xyz=0.00040486 -0.10983 0 rpy=1.5708 0 0
- joint joint6: limit lower=-3.14 upper=3.14 effort=100 velocity=1 -> lower=-2.96555 upper=2.96555 effort=100 velocity=1

File: GEN72/urdf/gen_72_b_description/urdf/GEN72.urdf (robot description, URDF)
Before this commit: robot GEN72, 8 links, 7 joints
Joints:
- joint joint6: limit lower=-1.707 upper=1.783 effort=5 velocity=3.141 -> lower=-1.600 upper=1.783 effort=5 velocity=3.141

File: RM65/urdf/rm_65_b_description/urdf/rm_65_b_description.urdf (robot description, URDF)
Before this commit: robot rm_65_b_description, 7 links, 6 joints
Links:
- link Link1: mass 0.59356 -> 0.593563443690403; geometry collision mesh filename=package://rm_65_b_description/meshes/link1.STL; visual mesh filename=package://rm_65_b_description/meshes/link1.STL
- link Link2: mass 0.86418 -> 0.864175046869043; geometry collision mesh filename=package://rm_65_b_description/meshes/link2.STL; visual mesh filename=package://rm_65_b_description/meshes/link2.STL
- link Link3: mass 0.28965 -> 0.289633681624654; geometry collision mesh filename=package://rm_65_b_description/meshes/link3.STL; visual mesh filename=package://rm_65_b_description/meshes/link3.STL
- link Link4: mass 0.23942 -> 0.239419768320061; geometry collision mesh filename=package://rm_65_b_description/meshes/link4.STL; visual mesh filename=package://rm_65_b_description/meshes/link4.STL
- link Link5: mass 0.21879 -> 0.218799761431678; geometry collision mesh filename=package://rm_65_b_description/meshes/link5.STL; visual mesh filename=package://rm_65_b_description/meshes/link5.STL
- link Link6: mass 0.065035 -> 0.0649018034311231; geometry collision mesh filename=package://rm_65_b_description/meshes/link6.STL; visual mesh filename=package://rm_65_b_description/meshes/link6.STL
- link base_link: mass 0.84108 -> 0.841070778135659
Joints:
- joint joint1: limit lower=-3.107 upper=3.107 effort=100 velocity=1 -> lower=-3.1 upper=3.1 effort=60 velocity=3.14
- joint joint2: limit lower=-2.269 upper=2.269 effort=100 velocity=1 -> lower=-2.268 upper=2.268 effort=60 velocity=3.14
- joint joint3: limit lower=-2.356 upper=2.356 effort=100 velocity=1 -> lower=-2.355 upper=2.355 effort=30 velocity=3.92
- joint joint4: limit lower=-3.107 upper=3.107 effort=100 velocity=1 -> lower=-3.1 upper=3.1 effort=10 velocity=3.92
- joint joint5: limit lower=-2.234 upper=2.234 effort=100 velocity=1 -> lower=-2.233 upper=2.233 effort=10 velocity=3.92
- joint joint6: limit lower=-6.283 upper=6.283 effort=100 velocity=1 -> lower=-6.28 upper=6.28 effort=10 velocity=3.92

File: RM75/urdf/rm_75_b_description/urdf/rm_75_b_description.urdf (robot description, URDF)
Before this commit: robot rm_75_b_description, 8 links, 7 joints
Links:
- link Link1: mass 0.59356 -> 0.593563458735581; geometry collision mesh filename=package://rm_75_b_description/meshes/link1.STL; visual mesh filename=package://rm_75_b_description/meshes/link1.STL
- link Link2: mass 0.43285 -> 0.432849770310974; geometry collision mesh filename=package://rm_75_b_description/meshes/link2.STL; visual mesh filename=package://rm_75_b_description/meshes/link2.STL
- link Link3: mass 0.43132 -> 0.431325495678459; geometry collision mesh filename=package://rm_75_b_description/meshes/link3.STL; visual mesh filename=package://rm_75_b_description/meshes/link3.STL
- link Link4: mass 0.289633678265103 -> 0.289633681619295; geometry collision mesh filename=package://rm_75_b_description/meshes/link4.STL; visual mesh filename=package://rm_75_b_description/meshes/link4.STL
- link Link5: mass 0.23941 -> 0.239419768320061; geometry collision mesh filename=package://rm_75_b_description/meshes/link5.STL; visual mesh filename=package://rm_75_b_description/meshes/link5.STL
- link Link6: mass 0.21879 -> 0.218799761431682; geometry collision mesh filename=package://rm_75_b_description/meshes/link6.STL; visual mesh filename=package://rm_75_b_description/meshes/link6.STL
- link Link7: mass 0.065035 -> 0.0649018034311231; geometry collision mesh filename=package://rm_75_b_description/meshes/link7.STL; visual mesh filename=package://rm_75_b_description/meshes/link7.STL
- link base_link: mass 0.84105 -> 0.841071174772543
Joints:
- joint joint1: limit lower=-3.107 upper=3.107 effort=100 velocity=1 -> lower=-3.1 upper=3.1 effort=60 velocity=3.14
- joint joint2: limit lower=-2.269 upper=2.269 effort=100 velocity=1 -> lower=-2.268 upper=2.268 effort=60 velocity=3.14
- joint joint3: limit lower=-3.107 upper=3.107 effort=100 velocity=1 -> lower=-3.1 upper=3.1 effort=30 velocity=3.92
- joint joint4: limit lower=-2.356 upper=2.356 effort=100 velocity=1 -> lower=-2.355 upper=2.355 effort=30 velocity=3.92
- joint joint5: limit lower=-3.107 upper=3.107 effort=100 velocity=1 -> lower=-3.1 upper=3.1 effort=10 velocity=3.92
- joint joint6: limit lower=-2.234 upper=2.234 effort=100 velocity=1 -> lower=-2.233 upper=2.233 effort=10 velocity=3.92
- joint joint7: limit lower=-6.283 upper=6.283 effort=100 velocity=1 -> lower=-6.28 upper=6.28 effort=10 velocity=3.92

File: RML63/urdf/rm_63_b_description/urdf/rm_63_b_description.urdf (robot description, URDF)
Before this commit: robot rm_63_b_description, 7 links, 6 joints
Links:
- removed link Link1
- removed link Link2
- removed link Link3
- removed link Link4
- removed link Link5
- removed link Link6
- added link link1, mass 0.89496; collision mesh filename=package://rm_63_b_description/meshes/link1.STL; visual mesh filename=package://rm_63_b_description/meshes/link1.STL
- added link link2, mass 1.5679; collision mesh filename=package://rm_63_b_description/meshes/link2.STL; visual mesh filename=package://rm_63_b_description/meshes/link2.STL
- added link link3, mass 0.67539; collision mesh filename=package://rm_63_b_description/meshes/link3.STL; visual mesh filename=package://rm_63_b_description/meshes/link3.STL
- added link link4, mass 0.69687; collision mesh filename=package://rm_63_b_description/meshes/link4.STL; visual mesh filename=package://rm_63_b_description/meshes/link4.STL
- added link link5, mass 0.34759; collision mesh filename=package://rm_63_b_description/meshes/link5.STL; visual mesh filename=package://rm_63_b_description/meshes/link5.STL
- added link link6, mass 0.077104; collision mesh filename=package://rm_63_b_description/meshes/link6.STL; visual mesh filename=package://rm_63_b_description/meshes/link6.STL
Joints:
- joint joint1: child Link1 -> link1; limit lower=-3.107 upper=3.107 effort=100 velocity=1 -> lower=-3.106 upper=3.106 effort=100 velocity=1
- joint joint2: child Link2 -> link2; limit lower=-3.107 upper=3.107 effort=100 velocity=1 -> lower=-3.106 upper=3.106 effort=100 velocity=1; origin xyz=-0.086 0 0 rpy=-1.5708 -1.5708 0 -> xyz=-0.086 0 0 rpy=0 -1.5708 -1.5708; parent Link1 -> link1
- joint joint3: child Link3 -> link3; limit lower=-3.107 upper=2.531 effort=100 velocity=1 -> lower=-3.106 upper=2.53 effort=100 velocity=1; parent Link2 -> link2
- joint joint4: child Link4 -> link4; limit lower=-3.107 upper=3.107 effort=100 velocity=1 -> lower=-3.106 upper=3.106 effort=100 velocity=1; origin xyz=0.067482 -0.405 -0.00051458 rpy=1.5708 0 0 -> xyz=0.069 -0.405 0.00029958 rpy=1.5708 0 0; parent Link3 -> link3
- joint joint5: child Link5 -> link5; limit lower=-3.107 upper=3.107 effort=100 velocity=1 -> lower=-3.106 upper=3.106 effort=100 velocity=1; parent Link4 -> link4
- joint joint6: child Link6 -> link6; limit lower=-6.283 upper=6.283 effort=100 velocity=1 -> lower=-6.28 upper=6.28 effort=100 velocity=1; origin xyz=-0.0015175 0.115 0.00081415 rpy=1.5708 0 3.1416 -> xyz=0 0.115 0 rpy=1.5708 0 3.1416; parent Link5 -> link5
