Commit message: doc:update GEN72 urdf

File: GEN72/urdf/gen_72_b_description/urdf/GEN72.urdf (robot description, URDF)
Before this commit: robot GEN72, 8 links, 7 joints
Links:
- link Link1: geometry collision mesh filename=package://rm_description/meshes/GEN72/Link1.STL; visual mesh filename=package://rm_description/meshes/GEN72/Link1.STL
- link Link2: geometry collision mesh filename=package://rm_description/meshes/GEN72/Link2.STL; visual mesh filename=package://rm_description/meshes/GEN72/Link2.STL
- link Link3: mass 0.774130450031732 -> 0.774130450031718; geometry collision mesh filename=package://rm_description/meshes/GEN72/Link3.STL; visual mesh filename=package://rm_description/meshes/GEN72/Link3.STL
- link Link4: mass 0.437130215853835 -> 0.437130215853825; geometry collision mesh filename=package://rm_description/meshes/GEN72/Link4.STL; visual mesh filename=package://rm_description/meshes/GEN72/Link4.STL
- link Link5: geometry collision mesh filename=package://rm_description/meshes/GEN72/Link5.STL; visual mesh filename=package://rm_description/meshes/GEN72/Link5.STL
- link Link6: geometry collision mesh filename=package://rm_description/meshes/GEN72/Link6.STL; visual mesh filename=package://rm_description/meshes/GEN72/Link6.STL
- link Link7: mass 0.127401822079286 -> 0.176612671882913; geometry collision mesh filename=package://rm_description/meshes/GEN72/Link7.STL; visual mesh filename=package://rm_description/meshes/GEN72/Link7.STL
- link base_link: mass 0.725732279372221 -> 0.725732279372378; geometry collision mesh filename=package://rm_description/meshes/GEN72/base_link.STL; visual mesh filename=package://rm_description/meshes/GEN72/base_link.STL
Joints:
- joint joint5: limit lower=-3.0014 upper=3.0014 effort=5 velocity=3.141 -> lower=-3.0014 upper=3.0014 effort=5 velocity=3.926
- joint joint6: limit lower=-1.600 upper=1.783 effort=5 velocity=3.141 -> lower=-1.707 upper=1.783 effort=5 velocity=3.926
- joint joint7: axis 0 1 0 -> 0 0 1; limit lower=-3.0014 upper=3.0014 effort=5 velocity=3.141 -> lower=-3.0014 upper=3.0014 effort=5 velocity=3.926; origin xyz=0.0742 0.067 0 rpy=0 0 1.5708 -> xyz=0.0905 0.067 0 rpy=1.5708 0 1.5708
