Commit message: 修改

File: RML63/urdf/RML63III/rm_63_b_description/urdf/RML-63.urdf (robot description, URDF)
Before this commit: robot RML-63, 7 links, 6 joints
Links:
- link Link_1: mass 1.76684172446222 -> 1.7668
- link Link_2: mass 4.34134499577628 -> 4.3415
- link Link_3: mass 1.72863066563727 -> 1.7286
- link Link_4: mass 2.47324011006769 -> 2.4734
- link Link_5: mass 0.931616551800953 -> 0.93162
- link Link_6: mass 0.305602476906259 -> 0.065037
- link base_link: mass 1.6314377241954 -> 1.6314
Joints:
- joint joint_4: origin xyz=0.06899998447855 -0.404999872232 0 rpy=1.5707963267949 0 0 -> xyz=0.069 -0.405 0 rpy=1.5708 0 0
- joint joint_5: origin xyz=0 0 0 rpy=1.5708 0 -3.1416 -> xyz=0 0 0 rpy=1.5708 0 3.1416
- joint joint_6: origin xyz=0 0.132199355735491 0 rpy=1.5708 0 -3.1416 -> xyz=-0.00010308 0.115 -0.00010734 rpy=1.5708 0 3.1416
