Commit message: docs: update the urdf files of RX75 and ECO62
Signed-off-by: rocky <rocky@realman-robot.com>

File: ECO62/urdf/ECO62-B/urdf/ECO62URDF.urdf (robot description, URDF)
Before this commit: robot ECO62URDF, 7 links, 6 joints
Links:
- link link_1: mass 0.384569120432882 -> 1.19575
- link link_2: mass 1.33623855048231 -> 0.8055
- link link_3: mass 0.332154099628179 -> 0.413
- link link_4: mass 0.110752178156894 -> 0.2386
- link link_5: mass 0.153716854003785 -> 0.2633
- link link_6: mass 0.0471960682349858 -> 0.0667
Joints:
- joint joint_2: axis 0 0 -1 -> 0 0 1; limit lower=-1.8151 upper=2.9496 effort=10 velocity=3.927 -> lower=-2.9496 upper=1.8151 effort=10 velocity=3.927
- joint joint_4: axis 0 0 -1 -> 0 0 1
- joint joint_6: axis 0 0 0.999999999999983 -> 0 0 1

File: RX75/urdf/RX75-6FB-V/RXL-6FB-V/urdf/RXL-6FB-V.urdf (robot description, URDF)
Before this commit: robot RXL-6F-C3, 9 links, 8 joints
Links:
- removed link Link2L
- added link Link2, mass 1.394; collision mesh filename=package://RXL-6FB-V/meshes/Link2.STL; visual mesh filename=package://RXL-6FB-V/meshes/Link2.STL
- link Link1: mass 0.851539025255045 -> 1.559; geometry collision mesh filename=package://RXL-6FB-V/meshes/Link1.STL; visual mesh filename=package://RXL-6FB-V/meshes/Link1.STL
- link Link3: mass 0.593225772794727 -> 1.117; geometry collision mesh filename=package://RXL-6FB-V/meshes/Link3.STL; visual mesh filename=package://RXL-6FB-V/meshes/Link3.STL
- link Link4: mass 0.395483521349425 -> 0.673; geometry collision mesh filename=package://RXL-6FB-V/meshes/Link4.STL; visual mesh filename=package://RXL-6FB-V/meshes/Link4.STL
- link Link5: mass 0.845200684581008 -> 1.13; geometry collision mesh filename=package://RXL-6FB-V/meshes/Link5.STL; visual mesh filename=package://RXL-6FB-V/meshes/Link5.STL
- link Link6: mass 0.28094 -> 0.559; geometry collision mesh filename=package://RXL-6FB-V/meshes/Link6.STL; visual mesh filename=package://RXL-6FB-V/meshes/Link6.STL
- link Link7: mass 0.163718739821727 -> 0.483; geometry collision mesh filename=package://RXL-6FB-V/meshes/Link7.STL; visual mesh filename=package://RXL-6FB-V/meshes/Link7.STL
- link Link8: geometry collision mesh filename=package://RXL-6FB-V/meshes/Link8.STL; visual mesh filename=package://RXL-6FB-V/meshes/Link8.STL
- link base_link: mass 0.651913537431336 -> 0.651913537431184; geometry collision mesh filename=package://RXL-6FB-V/meshes/base_link.STL; visual mesh filename=package://RXL-6FB-V/meshes/base_link.STL
Joints:
- removed joint J2L
- added joint J2: type revolute, parent Link1, child Link2, origin xyz=0 0 0 rpy=-1.57079632679489 -1.5707963267949 0, axis 0 0 1, limit lower=-0.6109 upper=3.1067 effort=60 velocity=3.14
- joint J1: axis 0 0 -1 -> 0 0 1; limit lower=-3.105 upper=3.105 effort=60 velocity=3.14 -> lower=-3.0194 upper=3.0194 effort=60 velocity=3.14
- joint J3: axis 0 0 -1 -> 0 0 1; limit lower=-3.105 upper=3.105 effort=30 velocity=3.925 -> lower=-3.0194 upper=3.0194 effort=30 velocity=3.925; parent Link2L -> Link2
- joint J4: axis 0 0 -1 -> 0 0 1; limit lower=-2.355 upper=2.355 effort=30 velocity=3.925 -> lower=-2.2689 upper=0.2618 effort=30 velocity=3.925
- joint J5: axis 0 0 -1 -> 0 0 1; limit lower=-3.105 upper=3.105 effort=10 velocity=3.925 -> lower=-3.0194 upper=3.0194 effort=10 velocity=3.925
- joint J6: axis 0 0 -1 -> 0 0 1; limit lower=-1.046 upper=1.046 effort=10 velocity=3.925 -> lower=-0.9599 upper=0.9599 effort=10 velocity=3.925; origin xyz=0 0 0 rpy=1.5708 -1.5708 0 -> xyz=0 0 0 rpy=1.57079632679489 -1.5707963267949 0
- joint J7: axis 0 0 -1 -> 0 0 1; limit lower=-1.988 upper=0.697 effort=10 velocity=3.925 -> lower=-1.9024 upper=0.6109 effort=10 velocity=3.925
- joint J8: axis 0 1 0 -> 0 0 1; origin xyz=0 -0.0962000041171294 0 rpy=1.57079632679489 0 0 -> xyz=0 -0.119000004117148 0 rpy=1.57079632679489 0 0

File: RX75/urdf/RX75-6FB-V/RXR-6FB-V/urdf/RXR-6FB-V.urdf (robot description, URDF)
Before this commit: robot RXR-6FB-V, 9 links, 8 joints
Links:
- link Link1: mass 0.851539173063523 -> 1.559
- link Link2: mass 0.87008 -> 1.384
- link Link3: mass 0.593225765910811 -> 1.117
- link Link4: mass 0.395483546701072 -> 0.665
- link Link5: mass 0.845201652493134 -> 1.13
- link Link6: mass 0.280941853294711 -> 0.559
- link Link7: mass 0.229769882476631 -> 0.483
Joints:
- joint J1: axis 0 0 -1 -> 0 0 1; limit lower=-0.785 upper=3.1 effort=60 velocity=3.14 -> lower=-3.0194 upper=3.0194 effort=60 velocity=3.14
- joint J2: limit lower=-0.524 upper=3.11 effort=60 velocity=3.14 -> lower=-0.6109 upper=3.1067 effort=60 velocity=3.14; origin xyz=0 0 0 rpy=1.5708 -1.5708 0 -> xyz=0 0 0 rpy=-1.5708 -1.5708 0
- joint J3: axis 0 0 -1 -> 0 0 1; limit lower=-3.11 upper=3.11 effort=30 velocity=3.925 -> lower=-3.0194 upper=3.0194 effort=30 velocity=3.925
- joint J4: limit lower=-2.62 upper=0 effort=30 velocity=3.925 -> lower=-2.2689 upper=0.2618 effort=30 velocity=3.925
- joint J5: axis 0 0 -1 -> 0 0 1; limit lower=-3.11 upper=3.11 effort=10 velocity=3.925 -> lower=-3.0194 upper=3.0194 effort=10 velocity=3.925
- joint J6: limit lower=-1.13 upper=1.13 effort=10 velocity=3.925 -> lower=-0.9599 upper=0.9599 effort=10 velocity=3.925
- joint J7: axis 0 0 -1 -> 0 0 1; limit lower=-0.697 upper=1.99 effort=10 velocity=3.925 -> lower=-0.6109 upper=1.9024 effort=10 velocity=3.925
- joint J8: axis 0 0 -1 -> 0 0 1; type revolute -> fixed

File: RX75/urdf/RX75-6FB/RXL-6F-C3/urdf/RXL-6F-C3.urdf (robot description, URDF)
Before this commit: robot RXR-6F-C3, 9 links, 8 joints
Links:
- removed link Link2
- added link Link2L, mass 1.394; collision mesh filename=package://RXL-6F-C3/meshes/Link2L.STL; visual mesh filename=package://RXL-6F-C3/meshes/Link2L.STL
- link Link1: mass 0.851539173063523 -> 1.559; geometry collision mesh filename=package://RXL-6F-C3/meshes/Link1.STL; visual mesh filename=package://RXL-6F-C3/meshes/Link1.STL
- link Link3: mass 0.593225765910811 -> 1.117; geometry collision mesh filename=package://RXL-6F-C3/meshes/Link3.STL; visual mesh filename=package://RXL-6F-C3/meshes/Link3.STL
- link Link4: mass 0.395483546755608 -> 0.673; geometry collision mesh filename=package://RXL-6F-C3/meshes/Link4.STL; visual mesh filename=package://RXL-6F-C3/meshes/Link4.STL
- link Link5: mass 0.845201652493134 -> 1.13; geometry collision mesh filename=package://RXL-6F-C3/meshes/Link5.STL; visual mesh filename=package://RXL-6F-C3/meshes/Link5.STL
- link Link6: mass 0.280941853294711 -> 0.559; geometry collision mesh filename=package://RXL-6F-C3/meshes/Link6.STL; visual mesh filename=package://RXL-6F-C3/meshes/Link6.STL
- link Link7: mass 0.16371 -> 0.483; geometry collision mesh filename=package://RXL-6F-C3/meshes/Link7.STL; visual mesh filename=package://RXL-6F-C3/meshes/Link7.STL
- link Link8: mass 0.165822947667674 -> 0.0; geometry collision mesh filename=package://RXL-6F-C3/meshes/Link8.STL; visual mesh filename=package://RXL-6F-C3/meshes/Link8.STL
- link base_link: mass 0.651913537431184 -> 0.651913537431336; geometry collision mesh filename=package://RXL-6F-C3/meshes/base_link.STL; visual mesh filename=package://RXL-6F-C3/meshes/base_link.STL
Joints:
- removed joint J2
- added joint J2L: type revolute, parent Link1, child Link2L, origin xyz=0 0 0 rpy=-1.57079632679489 -1.5707963267949 0, axis 0 0 1, limit lower=-0.6109 upper=3.1067 effort=60 velocity=3.14
- joint J1: axis 0 0 -1 -> 0 0 1; limit lower=-0.785 upper=3.1 effort=60 velocity=3.14 -> lower=-3.0194 upper=3.0194 effort=60 velocity=3.14; origin xyz=0 0 0.1915 rpy=0 0 0 -> xyz=0 0 0.191500058118611 rpy=0 0 0
- joint J3: axis 0 0 -1 -> 0 0 1; limit lower=-3.11 upper=3.11 effort=30 velocity=3.925 -> lower=-3.0194 upper=3.0194 effort=30 velocity=3.925; origin xyz=0 -0.322 0 rpy=1.5707963267949 1.5707963267949 0 -> xyz=0 -0.322 0 rpy=1.5707963267949 -1.5707963267949 0; parent Link2 -> Link2L
- joint J4: limit lower=-2.62 upper=0 effort=30 velocity=3.925 -> lower=-2.2689 upper=0.2618 effort=30 velocity=3.925
- joint J5: axis 0 0 -1 -> 0 0 1; limit lower=-3.11 upper=3.11 effort=10 velocity=3.925 -> lower=-3.0194 upper=3.0194 effort=10 velocity=3.925
- joint J6: limit lower=-1.13 upper=1.13 effort=10 velocity=3.925 -> lower=-0.9599 upper=0.9599 effort=10 velocity=3.925; origin xyz=0 0 0 rpy=1.5707963267949 -1.5707963267949 0 -> xyz=0 0 0 rpy=1.5708 -1.5708 0
- joint J7: axis 0 0 -1 -> 0 0 1; limit lower=-0.697 upper=1.99 effort=10 velocity=3.925 -> lower=-1.9024 upper=0.6109 effort=10 velocity=3.925; origin xyz=0.0155 0 0 rpy=1.5708 1.5708 0 -> xyz=0.0155 0 0 rpy=1.5708 -1.5708 0
- joint J8: axis 0 0 -1 -> 0 0 1; origin xyz=0 0.0962 0 rpy=-1.5708 0 0 -> xyz=0 -0.0962000041171294 0 rpy=1.57079632679489 0 0; type revolute -> fixed

File: RX75/urdf/RX75-6FB/RXR-6F-C3/urdf/RXR-6F-C3.urdf (robot description, URDF)
Before this commit: robot RXL-6FB-V, 9 links, 8 joints
Links:
- link Link1: mass 0.851539025255045 -> 1.559; geometry collision mesh filename=package://RXR-6F-C3/meshes/Link1.STL; visual mesh filename=package://RXR-6F-C3/meshes/Link1.STL
- link Link2: mass 0.870077465148622 -> 1.384; geometry collision mesh filename=package://RXR-6F-C3/meshes/Link2.STL; visual mesh filename=package://RXR-6F-C3/meshes/Link2.STL
- link Link3: mass 0.593225766113055 -> 1.117; geometry collision mesh filename=package://RXR-6F-C3/meshes/Link3.STL; visual mesh filename=package://RXR-6F-C3/meshes/Link3.STL
- link Link4: mass 0.395483565870343 -> 0.665; geometry collision mesh filename=package://RXR-6F-C3/meshes/Link4.STL; visual mesh filename=package://RXR-6F-C3/meshes/Link4.STL
- link Link5: mass 0.845200261498234 -> 1.13; geometry collision mesh filename=package://RXR-6F-C3/meshes/Link5.STL; visual mesh filename=package://RXR-6F-C3/meshes/Link5.STL
- link Link6: mass 0.280942850777542 -> 0.559; geometry collision mesh filename=package://RXR-6F-C3/meshes/Link6.STL; visual mesh filename=package://RXR-6F-C3/meshes/Link6.STL
- link Link7: mass 0.23898 -> 0.483; geometry collision mesh filename=package://RXR-6F-C3/meshes/Link7.STL; visual mesh filename=package://RXR-6F-C3/meshes/Link7.STL
- link Link8: mass 0.16582 -> 0.0; geometry collision mesh filename=package://RXR-6F-C3/meshes/Link8.STL; visual mesh filename=package://RXR-6F-C3/meshes/Link8.STL
- link base_link: geometry collision mesh filename=package://RXR-6F-C3/meshes/base_link.STL; visual mesh filename=package://RXR-6F-C3/meshes/base_link.STL
Joints:
- joint J1: axis 0 0 -1 -> 0 0 1; limit lower=-3.105 upper=3.105 effort=60 velocity=3.14 -> lower=-3.0194 upper=3.0194 effort=60 velocity=3.14; origin xyz=0 0 0.191500058118611 rpy=0 0 0 -> xyz=0 0 0.1915 rpy=0 0 0
- joint J2: limit lower=-0.697 upper=3.837 effort=60 velocity=3.14 -> lower=-0.6109 upper=3.1067 effort=60 velocity=3.14; origin xyz=0 0 0 rpy=1.57079632679489 -1.5707963267949 0 -> xyz=0 0 0 rpy=-1.57079632679489 -1.5707963267949 0
- joint J3: axis 0 0 -1 -> 0 0 1; limit lower=-3.105 upper=3.105 effort=30 velocity=3.925 -> lower=-3.0194 upper=3.0194 effort=30 velocity=3.925; origin xyz=0 -0.322 0 rpy=1.5707963267949 -1.5707963267949 0 -> xyz=0 -0.322 0 rpy=1.5707963267949 1.5707963267949 0
- joint J4: axis 0 0 -1 -> 0 0 1; limit lower=-2.355 upper=2.355 effort=30 velocity=3.925 -> lower=-2.2689 upper=0.2618 effort=30 velocity=3.925
- joint J5: axis 0 0 -1 -> 0 0 1; limit lower=-3.105 upper=3.105 effort=10 velocity=3.925 -> lower=-3.0194 upper=3.0194 effort=10 velocity=3.925
- joint J6: axis 0 0 -1 -> 0 0 1; limit lower=-1.046 upper=1.046 effort=10 velocity=3.925 -> lower=-0.9599 upper=0.9599 effort=10 velocity=3.925; origin xyz=0 0 0 rpy=1.57079632679489 -1.5707963267949 0 -> xyz=0 0 0 rpy=1.5707963267949 -1.5707963267949 0
- joint J7: axis 0 0 -1 -> 0 0 1; limit lower=-1.988 upper=0.697 effort=10 velocity=3.925 -> lower=-0.6109 upper=1.9024 effort=10 velocity=3.925; origin xyz=0.0155 0 0 rpy=1.5708 -1.5708 0 -> xyz=0.0155 0 0 rpy=1.5708 1.5708 0
- joint J8: axis 0 0 -1 -> 0 0 1; origin xyz=0 -0.119000004117148 0 rpy=1.57079632679489 0 0 -> xyz=0 0.0962 0 rpy=-1.5708 0 0; type revolute -> fixed
