Commit message: docs: update the urdf files of RX75
Signed-off-by: rocky <rocky@realman-robot.com>

File: RX75/urdf/RX75-B-V/RXL-B-V/urdf/RXL-B-V.urdf (robot description, URDF)
Before this commit: robot RXR-6FB-V, 9 links, 8 joints
Links:
- link Link1: geometry collision mesh filename=package://RXL-B-V/meshes/Link1.STL; visual mesh filename=package://RXL-B-V/meshes/Link1.STL
- link Link2: mass 1.384 -> 1.394; geometry collision mesh filename=package://RXL-B-V/meshes/Link2.STL; visual mesh filename=package://RXL-B-V/meshes/Link2.STL
- link Link3: geometry collision mesh filename=package://RXL-B-V/meshes/Link3.STL; visual mesh filename=package://RXL-B-V/meshes/Link3.STL
- link Link4: mass 0.665 -> 0.673; geometry collision mesh filename=package://RXL-B-V/meshes/Link4.STL; visual mesh filename=package://RXL-B-V/meshes/Link4.STL
- link Link5: geometry collision mesh filename=package://RXL-B-V/meshes/Link5.STL; visual mesh filename=package://RXL-B-V/meshes/Link5.STL
- link Link6: geometry collision mesh filename=package://RXL-B-V/meshes/Link6.STL; visual mesh filename=package://RXL-B-V/meshes/Link6.STL
- link Link7: mass 0.483 -> 0.433; geometry collision mesh filename=package://RXL-B-V/meshes/Link7.STL; visual mesh filename=package://RXL-B-V/meshes/Link7.STL
- link Link8: mass 0.165822947667674 -> 0.0696336896784389; geometry collision mesh filename=package://RXL-B-V/meshes/Link8.STL; visual mesh filename=package://RXL-B-V/meshes/Link8.STL
- link base_link: mass 0.651913537431336 -> 0.651913537431335; geometry collision mesh filename=package://RXL-B-V/meshes/base_link.STL; visual mesh filename=package://RXL-B-V/meshes/base_link.STL
Joints:
- joint J1: origin xyz=0 0 0.1915 rpy=0 0 0 -> xyz=0 0 0.191500058118611 rpy=0 0 0
- joint J2: origin xyz=0 0 0 rpy=-1.5708 -1.5708 0 -> xyz=0 0 0 rpy=-1.57079632679489 -1.5707963267949 0
- joint J3: origin xyz=0 -0.322 0 rpy=1.5707963267949 1.5707963267949 0 -> xyz=0 -0.322 0 rpy=1.5708 -1.5708 0
- joint J6: origin xyz=0 0 0 rpy=1.5707963267949 -1.5707963267949 0 -> xyz=0 0 0 rpy=1.57079632679489 -1.5707963267949 0
- joint J7: limit lower=-0.6109 upper=1.9024 effort=10 velocity=3.925 -> lower=-1.9024 upper=0.6109 effort=10 velocity=3.925; origin xyz=0.0155 0 0 rpy=1.5708 1.5708 0 -> xyz=0.0155 0 0 rpy=1.57079632679489 -1.5707963267949 0
- joint J8: origin xyz=0 0.119000004117148 0 rpy=-1.5707963267949 0 0 -> xyz=0.000150519230103341 -0.101800004117148 -0.00015051923075171 rpy=1.57079632679489 0 0

File: RX75/urdf/RX75-B-V/RXR-B-V/urdf/RXR-B-V.urdf (robot description, URDF)
Before this commit: robot RXR-6FB-V, 9 links, 8 joints
Links:
- link Link1: geometry collision mesh filename=package://RXR-B-V/meshes/Link1.STL; visual mesh filename=package://RXR-B-V/meshes/Link1.STL
- link Link2: geometry collision mesh filename=package://RXR-B-V/meshes/Link2.STL; visual mesh filename=package://RXR-B-V/meshes/Link2.STL
- link Link3: geometry collision mesh filename=package://RXR-B-V/meshes/Link3.STL; visual mesh filename=package://RXR-B-V/meshes/Link3.STL
- link Link4: geometry collision mesh filename=package://RXR-B-V/meshes/Link4.STL; visual mesh filename=package://RXR-B-V/meshes/Link4.STL
- link Link5: geometry collision mesh filename=package://RXR-B-V/meshes/Link5.STL; visual mesh filename=package://RXR-B-V/meshes/Link5.STL
- link Link6: geometry collision mesh filename=package://RXR-B-V/meshes/Link6.STL; visual mesh filename=package://RXR-B-V/meshes/Link6.STL
- link Link7: geometry collision mesh filename=package://RXR-B-V/meshes/Link7.STL; visual mesh filename=package://RXR-B-V/meshes/Link7.STL
- link Link8: mass 0.165822947667674 -> 0.0696336896784392; geometry collision mesh filename=package://RXR-B-V/meshes/Link8.STL; visual mesh filename=package://RXR-B-V/meshes/Link8.STL
- link base_link: geometry collision mesh filename=package://RXR-B-V/meshes/base_link.STL; visual mesh filename=package://RXR-B-V/meshes/base_link.STL
Joints:
- joint J2: origin xyz=0 0 0 rpy=-1.5708 -1.5708 0 -> xyz=0 0 0 rpy=-1.57079632679489 -1.5707963267949 0
- joint J8: origin xyz=0 0.119000004117148 0 rpy=-1.5707963267949 0 0 -> xyz=0.000150519230103591 0.101800004117148 0.00015051923068905 rpy=-1.5707963267949 0 0
