Commit message: fix: Fix abnormal link inertia parameters in the URDF file of RX75
Signed-off-by: rocky <rocky@realman-robot.com>

File: RX75/urdf/RX75-6FB-V/RXL-6FB-V/urdf/RXL-6FB-V.urdf (robot description, URDF)
Before this commit: robot RXL-6FB-V, 9 links, 8 joints
Links:
- link Link8: mass 0.16582 -> 0
- link base_link: mass 0.651913537431184 -> 1.36

File: RX75/urdf/RX75-6FB-V/RXR-6FB-V/urdf/RXR-6FB-V.urdf (robot description, URDF)
Before this commit: robot RXR-6FB-V, 9 links, 8 joints
Links:
- link Link8: mass 0.165822947667674 -> 0
- link base_link: mass 0.651913537431336 -> 1.36

File: RX75/urdf/RX75-6FB/RXL-6F-C3/urdf/RXL-6F-C3.urdf (robot description, URDF)
Before this commit: robot RXL-6F-C3, 9 links, 8 joints
Links:
- link base_link: mass 0.651913537431336 -> 1.360

File: RX75/urdf/RX75-6FB/RXR-6F-C3/urdf/RXR-6F-C3.urdf (robot description, URDF)
Before this commit: robot RXR-6F-C3, 9 links, 8 joints
Links:
- link base_link: mass 0.651913537431184 -> 1.360

File: RX75/urdf/RX75-B-V/RXL-B-V/urdf/RXL-B-V.urdf (robot description, URDF)
Before this commit: robot RXL-B-V, 9 links, 8 joints
Links:
- link Link8: mass 0.0696336896784389 -> 0
- link base_link: mass 0.651913537431335 -> 1.36

File: RX75/urdf/RX75-B-V/RXR-B-V/urdf/RXR-B-V.urdf (robot description, URDF)
Before this commit: robot RXR-B-V, 9 links, 8 joints
Links:
- link Link7: mass 0.483 -> 0.433
- link Link8: mass 0.0696336896784392 -> 0
- link base_link: mass 0.651913537431336 -> 1.36
